File: guarduino_power.kicad_pcb (KiCad board)
At the start: 2 copper layers, 98.4 x 48.3 mm, 22 parts, among them K1 RELAY, P1 3way terminal, P2 3way terminal, P3 4way connector, T1 5V/1W

Commit message: Final production board
Parts:
- added REF**: Symbol_Highvoltage_Type1_CopperTop_Small, Symbols:Symbol_Highvoltage_Type1_CopperTop_Small, B.Cu at (55.9, 81.3)
- added REF**: Symbol_Highvoltage_Type1_CopperTop_Small, Symbols:Symbol_Highvoltage_Type1_CopperTop_Small, B.Cu at (83.8, 50.8)
Other:
- board text added: "GUARDUINO POWER SUPPLY ver 1.0, Jakub Nedbal 2016, CC-BY-SA"
- board text removed: "RAINING CATS POWER SUPPLY ver 1.0, Jakub Nedbal 2016, CC-BY-SA"
Changed lines of the file:
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@@
     (links 22)
     (no_connects 0)
-    (area 40.564999 40.564999 141.055944 89.945)
+    (area 40.564999 40.564999 139.140001 88.975001)
     (thickness 1.6)
     (drawings 48)
     (tracks 61)
     (zones 0)
-    (modules 22)
+    (modules 24)
     (nets 17)
   )
   (page A4)
   (title_block
-    (title "Raining Cats Power Supply")
+    (title "Guarduino Power Supply")
     (date 2016-09-25)
     (rev 1.0)
@@
     (add_net VCC)
   )
+  (module Symbols:Symbol_Highvoltage_Type1_CopperTop_Small (layer B.Cu)
+    (at 55.88 81.28 180)
+    (descr "Symbol, Highvoltage, Type 1, Copper Top, Small,")
+    (tags "Symbol, Highvoltage, Type 1, Copper Top, Small,")
+    (fp_text reference REF** (at 1.016 5.207 180) (layer B.SilkS) hide
+      (effects (font (size 1 1) (thickness 0.15)) (justify mirror))
+    )
+    (fp_text value Symbol_Highvoltage_Type1_CopperTop_Small (at 0.508 -4.191 180) (layer B.Fab) hide
+      (effects (font (size 1 1) (thickness 0.15)) (justify mirror))
+    )
+    (fp_line (start -0.381 0.762) (end 1.27 3.2385) (layer B.SilkS) (width 0.381))
+    (fp_line (start 1.27 3.2385) (end 1.397 2.794) (layer B.SilkS) (width 0.381))
+    (fp_line (start 1.397 2.794) (end 0 1.016) (layer B.SilkS) (width 0.381))
+    (fp_line (start 0 1.016) (end 1.143 0.889) (layer B.SilkS) (width 0.381))
+    (fp_line (start 2.159 3.175) (end 0.381 1.143) (layer B.SilkS) (width 0.381))
+    (fp_line (start 0.381 1.143) (end 1.651 1.143) (layer B.SilkS) (width 0.381))
+    (fp_line (start 2.159 3.175) (end 1.397 2.667) (layer B.SilkS) (width 0.381))
+    (fp_line (start -0.381 0.762) (end 1.016 0.762) (layer B.SilkS) (width 0.381))
+    (fp_line (start 1.016 0.762) (end -0.254 -1.778) (layer B.SilkS) (width 0.381))
+    (fp_line (start -0.127 -1.651) (end 1.651 1.143) (layer B.SilkS) (width 0.381))
+    (fp_line (start -0.254 -1.016) (end -0.381 -2.032) (layer B.SilkS) (width 0.381))
+    (fp_line (start -0.381 -2.032) (end 0.381 -1.397) (layer B.SilkS) (width 0.381))
+  )
+  (module Symbols:Symbol_Highvoltage_Type1_CopperTop_Small (layer B.Cu)
+    (at 83.82 50.8 180)
+    (descr "Symbol, Highvoltage, Type 1, Copper Top, Small,")
+    (tags "Symbol, Highvoltage, Type 1, Copper Top, Small,")
+    (fp_text reference REF** (at 1.016 5.207 180) (layer B.SilkS) hide
+      (effects (font (size 1 1) (thickness 0.15)) (justify mirror))
+    )
+    (fp_text value Symbol_Highvoltage_Type1_CopperTop_Small (at 0.508 -4.191 180) (layer B.Fab) hide
+      (effects (font (size 1 1) (thickness 0.15)) (justify mirror))
+    )
+    (fp_line (start -0.381 0.762) (end 1.27 3.2385) (layer B.SilkS) (width 0.381))
+    (fp_line (start 1.27 3.2385) (end 1.397 2.794) (layer B.SilkS) (width 0.381))
+    (fp_line (start 1.397 2.794) (end 0 1.016) (layer B.SilkS) (width 0.381))
+    (fp_line (start 0 1.016) (end 1.143 0.889) (layer B.SilkS) (width 0.381))
+    (fp_line (start 2.159 3.175) (end 0.381 1.143) (layer B.SilkS) (width 0.381))
+    (fp_line (start 0.381 1.143) (end 1.651 1.143) (layer B.SilkS) (width 0.381))
+    (fp_line (start 2.159 3.175) (end 1.397 2.667) (layer B.SilkS) (width 0.381))
+    (fp_line (start -0.381 0.762) (end 1.016 0.762) (layer B.SilkS) (width 0.381))
+    (fp_line (start 1.016 0.762) (end -0.254 -1.778) (layer B.SilkS) (width 0.381))
+    (fp_line (start -0.127 -1.651) (end 1.651 1.143) (layer B.SilkS) (width 0.381))
+    (fp_line (start -0.254 -1.016) (end -0.381 -2.032) (layer B.SilkS) (width 0.381))
+    (fp_line (start -0.381 -2.032) (end 0.381 -1.397) (layer B.SilkS) (width 0.381))
+  )
   (module Symbols:Symbol_Highvoltage_Type1_CopperTop_Small (layer F.Cu)
     (at 62.992 83.312)
@@
       (effects (font (size 1 1) (thickness 0.15)))
     )
-    (fp_text value Symbol_Highvoltage_Type1_CopperTop_Small (at 0.508 4.191) (layer F.Fab)
+    (fp_text value Symbol_Highvoltage_Type1_CopperTop_Small (at 0.508 4.191) (layer F.Fab) hide
       (effects (font (size 1 1) (thickness 0.15)))
     )
@@
       (effects (font (size 1 1) (thickness 0.15)))
     )
-    (fp_text value Symbol_Highvoltage_Type1_CopperTop_Small (at 0.508 4.191) (layer F.Fab)
+    (fp_text value Symbol_Highvoltage_Type1_CopperTop_Small (at 0.508 4.191) (layer F.Fab) hide
       (effects (font (size 1 1) (thickness 0.15)))
     )
@@
     (fp_line (start 0.74944 2.5003) (end 0.15 2.59936) (layer B.Cu) (width 0.381))
   )
-  (gr_text "RAINING CATS POWER SUPPLY ver 1.0, Jakub Nedbal 2016, CC-BY-SA" (at 89.662 87.122) (layer B.SilkS)
+  (gr_text "GUARDUINO POWER SUPPLY ver 1.0, Jakub Nedbal 2016, CC-BY-SA" (at 89.662 87.122) (layer B.SilkS)
     (effects (font (size 1.5 1.5) (thickness 0.3)) (justify mirror))
   )
@@
   )
   (gr_line (start 133.096 44.704) (end 46.736 44.704) (angle 90) (layer B.SilkS) (width 0.4))
-  (gr_text "RAINING CATS POWER SUPPLY ver 1.0, Jakub Nedbal 2016, CC-BY-SA" (at 89.535 86.995) (layer F.SilkS)
+  (gr_text "GUARDUINO POWER SUPPLY ver 1.0, Jakub Nedbal 2016, CC-BY-SA" (at 89.535 86.995) (layer F.SilkS)
     (effects (font (size 1.5 1.5) (thickness 0.3)))
   )
