File: guarduino_power.sch (KiCad schematic (older format))
At the start: 17 parts, among them K1 RELAY, P1 3way terminal, P2 3way terminal, P3 4way connector, T1 5V/1W

Commit message: Final production board
Parts:
- P3: Supplier Open parts library -> Open Parts Library
Other:
- note added: "HIGH CURRENT POWER SUPPLY SWITCH"
- note added: "LOW POWER AC/DC CONVERTER"
Changed lines of the file:
@@
 LIBS:valves
 LIBS:jakub
-LIBS:garduino_power-cache
+LIBS:guarduino_power-cache
 EELAYER 25 0
 EELAYER END
@@
 encoding utf-8
 Sheet 1 1
-Title "Raining Cats Power Supply"
+Title "Guarduino Power Supply"
 Date "2016-09-24"
 Rev "1.0"
 Comp "Serious Play Ltd"
 Comment1 "Jakub Nedbal"
-Comment2 ""
+Comment2 "License: CC-BY-SA"
 Comment3 ""
 Comment4 ""
@@
 F 5 "Taifeng" H 7650 2150 60  0001 C CNN "Manufacturer"
 F 6 "SIP-4" H 7650 2150 60  0001 C CNN "Package"
-F 7 "Open parts library" H 7650 2150 60  0001 C CNN "Supplier"
+F 7 "Open Parts Library" H 7650 2150 60  0001 C CNN "Supplier"
 F 8 "320110033" H 7650 2150 60  0001 C CNN "Order Code"
 F 9 "Farnell" H 7650 2150 60  0001 C CNN "Alt. Supplier"
@@
 Text Label 5300 2000 0    60   ~ 0
 NEUTRAL
-Text Notes 2900 4050 0    60   ~ 0
+Text Notes 2800 4050 0    60   ~ 0
 MOUNTING HOLES
 Text Notes 7850 2375 0    60   ~ 0
@@
 Text Notes 1300 3500 0    60   ~ 0
 5MM TERMINAL BLOCK\nConnect to external\npower supply\n230 VAC output
+Text Notes 5600 1500 0    60   ~ 0
+LOW POWER AC/DC CONVERTER
+Text Notes 3900 4400 0    60   ~ 0
+HIGH CURRENT POWER SUPPLY SWITCH
 $EndSCHEMATC
